Commit message: Update URDF with all the sensors and new bunker mini model

File: ros2_ws/bunker_description/urdf/bunker.urdf.xacro (robot description, xacro)
@@ -1,62 +1,24 @@
 <?xml version="1.0" encoding="utf-8"?>
 <!-- This URDF was automatically created by SolidWorks to URDF Exporter! Originally created by Stephen Brawner (brawner@gmail.com)
-     Commit Version: 1.6.0-1-g15f4949  Build Version: 1.6.7594.29634
+     Commit Version: 1.6.0-4-g7f85cfe  Build Version: 1.6.7995.38578
      For more information, please see http://wiki.ros.org/sw_urdf_exporter -->
-<robot  name="bunker_description" xmlns:xacro="http://www.ros.org/wiki/xacro">
+<robot
+  name="bunker_mini" xmlns:xacro="http://www.ros.org/wiki/xacro">
+  <xacro:include filename="sensors.urdf.xacro" />
   <link
     name="base_link">
-     <inertial>
+    <inertial>
       <origin
-        xyz="0.0212410555532523 0.00475458359568469 -0.127580557949736"
+        xyz="0.00266149933171387 -6.51753880652126E-06 -0.0988540390646707"
         rpy="0 0 0" />
       <mass
-        value="22" />
+        value="40.9538420525263" />
       <inertia
-        ixx="0.607716166684979"
-        ixy="1.92178193996147E-05"
-        ixz="-0.036532069356182"
-        iyy="1.70041426855404"
-        iyz="2.16963122007266E-05"
-        izz="1.84232351935185" />
-    </inertial>
-    <visual>
-      <origin
-        xyz="0.53 -0.392 -0.358"
-        rpy="1.57 0 3.14" />
-      <geometry>
-        <mesh
-          filename="package://bunker_description/meshes/BUNKER.STL" scale="0.001 0.001 0.001" />
-      </geometry>
-      <material
-        name="">
-        <color
-          rgba="0.5 0.5 0.5  1" />
-      </material>
-    </visual>
-    <collision>
-      <origin
-        xyz="0.53 -0.392 -0.358"
-        rpy="1.57 0 3.14" />
-      <geometry>
-        <mesh
-          filename="package://bunker_description/meshes/BUNKER.STL" scale="0.001 0.001 0.001" />
-      </geometry>
-    </collision>
-  </link>
-  <link
-    name="wheel1_Link">
-    <inertial>
-      <origin
-        xyz="0 -1.38777878078145E-17 -0.0719999999999999"
-        rpy="0 0 0" />
-      <mass
-        value="0.392034219968119" />
-      <inertia
-        ixx="0.000378440530116381"
-        ixy="5.60822736805661E-21"
-        ixz="3.04207802822425E-20"
-        iyy="0.000378440530116381"
-        iyz="-7.56626980356474E-21"
-        izz="0.000710150518820894" />
+        ixx="0.428867306980697"
+        ixy="-5.34500607982249E-06"
+        ixz="-0.0281290917935353"
+        iyy="1.22745608718324"
+        iyz="-7.8205947442509E-07"
+        izz="1.37929953930289" />
     </inertial>
     <visual>
@@ -66,5 +28,5 @@
       <geometry>
         <mesh
-          filename="package://bunker_description/meshes/wheel1_Link.STL" />
+          filename="package://bunker_description/meshes/base_link.STL" />
       </geometry>
       <material
@@ -80,895 +42,7 @@
       <geometry>
         <mesh
-          filename="package://bunker_description/meshes/wheel1_Link.STL" />
+          filename="package://bunker_description/meshes/base_link.STL" />
       </geometry>
     </collision>
   </link>
-  <joint
-    name="wheel1_joint"
-    type="revolute">
-    <origin
-      xyz="0.44403 0.3495 -0.12853"
-      rpy="1.5708 0 -3.1416" />
-    <parent
-      link="base_link" />
-    <child
-      link="wheel1_Link" />
-    <axis
-      xyz="0 0 1" />
-    <limit
-      lower="-180"
-      upper="180"
-      effort="0"
-      velocity="0" />
-  </joint>
-  <link
-    name="wheel1.1_Link">
-    <inertial>
-      <origin
-        xyz="-1.74279013442913E-08 5.87093572021469E-08 -0.0720000000000001"
-        rpy="0 0 0" />
-      <mass
-        value="0.190328287901002" />
-      <inertia
-        ixx="6.58750963981394E-05"
-        ixy="-1.46558944641469E-09"
-        ixz="-8.34967331718859E-12"
-        iyy="6.58795984671517E-05"
-        iyz="-2.4786046130206E-12"
-        izz="0.000112721820875598" />
-    </inertial>
-    <visual>
-      <origin
-        xyz="0 0 0"
-        rpy="0 0 0" />
-      <geometry>
-        <mesh
-          filename="package://bunker_description/meshes/wheel1.1_Link.STL" />
-      </geometry>
-      <material
-        name="">
-        <color
-          rgba="1 1 1 1" />
-      </material>
-    </visual>
-    <collision>
-      <origin
-        xyz="0 0 0"
-        rpy="0 0 0" />
-      <geometry>
-        <mesh
-          filename="package://bunker_description/meshes/wheel1.1_Link.STL" />
-      </geometry>
-    </collision>
-  </link>
-  <joint
-    name="wheel1.1_jont"
-    type="revolute">
-    <origin
-      xyz="0.37551 0.3495 -0.22305"
-      rpy="1.5708 0 -3.1416" />
-    <parent
-      link="base_link" />
-    <child
-      link="wheel1.1_Link" />
-    <axis
-      xyz="0 0 1" />
-    <limit
-      lower="-180"
-      upper="180"
-      effort="0"
-      velocity="0" />
-  </joint>
-  <link
-    name="wheel1.2_Link">
-    <inertial>
-      <origin
-        xyz="1.66533453693773E-16 4.16333634234434E-17 -0.0720000000000002"
-        rpy="0 0 0" />
-      <mass
-        value="0.271192811687251" />
-      <inertia
-        ixx="0.000179574259018481"
-        ixy="1.15789498120549E-20"
-        ixz="1.3563351843978E-21"
-        iyy="0.000179574259018481"
-        iyz="6.0369822309622E-23"
-        izz="0.000332594534732139" />
-    </inertial>
-    <visual>
-      <origin
-        xyz="0 0 0"
-        rpy="0 0 0" />
-      <geometry>
-        <mesh
-          filename="package://bunker_description/meshes/wheel1.2_Link.STL" />
-      </geometry>
-      <material
-        name="">
-        <color
-          rgba="1 1 1 1" />
-      </material>
-    </visual>
-    <collision>
-      <origin
-        xyz="0 0 0"
-        rpy="0 0 0" />
-      <geometry>
-        <mesh
-          filename="package://bunker_description/meshes/wheel1.2_Link.STL" />
-      </geometry>
-    </collision>
-  </link>
-  <joint
-    name="wheel1.2_joint"
-    type="revolute">
-    <origin
-      xyz="0.29039 0.3495 -0.28104"
-      rpy="1.5708 0 -3.1416" />
-    <parent
-      link="base_link" />
-    <child
-      link="wheel1.2_Link" />
-    <axis
-      xyz="0 0 1" />
-    <limit
-      lower="-180"
-      upper="180"
-      effort="0"
-      velocity="0" />
-  </joint>
-  <link
-    name="wheel1.3_Link">
-    <inertial>
-      <origin
-        xyz="3.44025652177504E-05 -2.66346274915008E-05 -0.0701504149473696"
-        rpy="0 0 0" />
-      <mass
-        value="0.245835028330933" />
-      <inertia
-        ixx="0.000105254202004996"
-        ixy="1.32328029886322E-08"
-        ixz="3.84294589102693E-11"
-        iyy="0.000105248656147198"
-        iyz="-1.41155611914915E-11"
-        izz="0.000173280771745758" />
-    </inertial>
-    <visual>
-      <origin
-        xyz="0 0 0"
-        rpy="0 0 0" />
-      <geometry>
-        <mesh
-          filename="package://bunker_description/meshes/wheel1.3_Link.STL" />
-      </geometry>
-      <material
-        name="">
-        <color
-          rgba="1 1 1 1" />
-      </material>
-    </visual>
-    <collision>
-      <origin
-        xyz="0 0 0"
-        rpy="0 0 0" />
-      <geometry>
-        <mesh
-          filename="package://bunker_description/meshes/wheel1.3_Link.STL" />
-      </geometry>
-    </collision>
-  </link>
-  <joint
-    name="wheel1.3_joint"
-    type="revolute">
-    <origin
-      xyz="0.29603 0.3495 -0.087"
-      rpy="1.5708 0 -3.1416" />
-    <parent
-      link="base_link" />
-    <child
-      link="wheel1.3_Link" />
-    <axis
-      xyz="0 0 -1" />
-    <limit
-      lower="-180"
-      upper="180"
-      effort="0"
-      velocity="0" />
-  </joint>
-  <link
-    name="wheel2_Link">
-    <inertial>
-      <origin
-        xyz="-1.66533453693773E-16 0 0.072"
-        rpy="0 0 0" />
-      <mass
-        value="0.392034219968119" />
-      <inertia
-        ixx="0.000378440530116381"
-        ixy="3.37302217863781E-21"
-        ixz="2.71827270955143E-20"
-        iyy="0.000378440530116381"
-        iyz="-7.32821644893157E-21"
-        izz="0.000710150518820894" />
-    </inertial>
-    <visual>
-      <origin
-        xyz="0 0 0"
-        rpy="0 0 0" />
-      <geometry>
-        <mesh
-          filename="package://bunker_description/meshes/wheel2_Link.STL" />
-      </geometry>
-      <material
-        name="">
-        <color
-          rgba="1 1 1 1" />
-      </material>
-    </visual>
-    <collision>
-      <origin
-        xyz="0 0 0"
-        rpy="0 0 0" />
-      <geometry>
-        <mesh
-          filename="package://bunker_description/meshes/wheel2_Link.STL" />
-      </geometry>
-    </collision>
-  </link>
-  <joint
-    name="wheel2_joint"
-    type="revolute">
-    <origin
-      xyz="0.44403 -0.3495 -0.12853"
-      rpy="1.5708 0 -3.1416" />
-    <parent
-      link="base_link" />
-    <child
-      link="wheel2_Link" />
-    <axis
-      xyz="0 0 -1" />
-    <limit
-      lower="-180"
-      upper="180"
-      effort="0"
-      velocity="0" />
-  </joint>
-  <link
-    name="wheel2.1_Link">
-    <inertial>
-      <origin
-        xyz="-1.74279017328693E-08 5.87093572160247E-08 0.0720000000000002"
-        rpy="0 0 0" />
-      <mass
-        value="0.190328287901002" />
-      <inertia
-        ixx="6.58750963981394E-05"
-        ixy="-1.46558944642761E-09"
-        ixz="-8.34967332343028E-12"
-        iyy="6.58795984671517E-05"
-        iyz="-2.47860459929511E-12"
-        izz="0.000112721820875598" />
-    </inertial>
-    <visual>
-      <origin
-        xyz="0 0 0"
-        rpy="0 0 0" />
-      <geometry>
-        <mesh
-          filename="package://bunker_description/meshes/wheel2.1_Link.STL" />
-      </geometry>
-      <material
-        name="">
-        <color
-          rgba="1 1 1 1" />
-      </material>
-    </visual>
-    <collision>
-      <origin
-        xyz="0 0 0"
-        rpy="0 0 0" />
-      <geometry>
-        <mesh
-          filename="package://bunker_description/meshes/wheel2.1_Link.STL" />
-      </geometry>
-    </collision>
-  </link>
-  <joint
-    name="wheel2.1_joint"
-    type="revolute">
-    <origin
-      xyz="0.37551 -0.3495 -0.22305"
-      rpy="1.5708 0 -3.1416" />
-    <parent
-      link="base_link" />
-    <child
-      link="wheel2.1_Link" />
-    <axis
-      xyz="0 0 -1" />
-    <limit
-      lower="-180"
-      upper="180"
-      effort="0"
-      velocity="0" />
-  </joint>
-  <link
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