Commit message: Update OAK TF in URDF. Change foxglove container to visualizer. Add calibration tools to visualizer container.

File: ros2_ws/bunker_description/urdf/sensors.urdf.xacro (robot description, xacro)
@@ -81,5 +81,5 @@
         </visual>
     </link>
-    <link name="25085490_qt128光罩_v2_0a0">
+    <link name="hesai_lidar">
         <inertial>
             <mass value="3.54543e-05" />
@@ -113,5 +113,5 @@
         </visual>
     </link>
-    <link name="502_mfp0044">
+    <link name="radar_1">
         <inertial>
             <mass value="2.93529e-05" />
@@ -421,5 +421,5 @@
         </visual>
     </link>
-    <link name="atlas_pre_dv_no_fov_110524">
+    <link name="aeva/vehicle">
         <inertial>
             <mass value="0.000581481" />
@@ -565,5 +565,5 @@
         </visual>
     </link>
-    <link name="d_pro_w_glass_lens_1">
+    <link name="oak_parent_frame">
         <inertial>
             <mass value="1.52404e-06" />
@@ -581,5 +581,5 @@
         </visual>
     </link>
-    <link name="d_pro_w_lens_adhesive_1">
+    <link name="oak">
         <inertial>
             <mass value="3.51525e-07" />
@@ -1188,5 +1188,5 @@
         </visual>
     </link>
-    <link name="sma_to_mcx_adapter_shell_aliner_20180924">
+    <link name="gps">
         <inertial>
             <mass value="2.81898e-07" />
@@ -1284,5 +1284,5 @@
         </visual>
     </link>
-    <link name="top_housing_mti_630r_casted_3_mti_630r_mti_6x0r_simple_2__mti_6x0r_simple">
+    <link name="imu">
         <inertial>
             <mass value="1.1973e-05" />
@@ -1362,5 +1362,5 @@
         <axis xyz="0 -1 0" />
         <parent link="part_5" />
-        <child link="atlas_pre_dv_no_fov_110524" />
+        <child link="aeva/vehicle" />
     </joint>
     <joint name="fastened_4" type="fixed">
@@ -1398,5 +1398,5 @@
         <axis xyz="0 0 1" />
         <parent link="502_mfm0572" />
-        <child link="502_mfp0044" />
+        <child link="radar_1" />
     </joint>
     <joint name="group_1_fastened_joint_1" type="fixed">
@@ -1488,5 +1488,5 @@
         <axis xyz="0 0 1" />
         <parent link="_mti_6x0r_simple_2__mti_6x0r_simple_5" />
-        <child link="top_housing_mti_630r_casted_3_mti_630r_mti_6x0r_simple_2__mti_6x0r_simple" />
+        <child link="imu" />
     </joint>
     <joint name="group_1_fastened_joint_23" type="fixed">
@@ -1662,5 +1662,5 @@
         <axis xyz="0 0 1" />
         <parent link="m2_5_insert_for_helix_family" />
-        <child link="sma_to_mcx_adapter_shell_aliner_20180924" />
+        <child link="gps" />
     </joint>
     <joint name="group_1_fastened_joint_5" type="fixed">
@@ -1686,5 +1686,5 @@
         <axis xyz="0 0 1" />
         <parent link="cable_spacer" />
-        <child link="d_pro_w_glass_lens_1" />
+        <child link="oak_parent_frame" />
     </joint>
     <joint name="group_1_fastened_joint_53" type="fixed">
@@ -1748,9 +1748,62 @@
         <child link="602_00007_1_1" />
     </joint>
+    <!--OAK-D-W Camera-->
     <joint name="group_1_fastened_joint_62" type="fixed">
-        <origin xyz="0 0 0" rpy="0 -0 0" />
-        <axis xyz="0 0 1" />
-        <parent link="d_pro_w_glass_lens_1" />
-        <child link="d_pro_w_lens_adhesive_1" />
+        <origin xyz="0 0 0" rpy="0 0 1.57" />
+        <axis xyz="0 0 1" />
+        <parent link="oak_parent_frame" />
+        <child link="oak" />
+    </joint>
+    <link name="oak_model_origin" />
+    <joint name="oak_model_origin_joint" type="fixed">
+        <parent link="oak" />
+        <child link="oak_model_origin" />
+        <origin xyz="0 0 0" rpy="1.5708 0 1.5708" />
+    </joint>
+    <link name="oak_imu_frame" />
+    <joint name="oak_imu_joint" type="fixed">
+        <parent link="oak" />
+        <child link="oak_imu_frame" />
+        <origin xyz="0.0 -0.015 -0.013662"
+            rpy="0.0 1.57 0.0" />
+    </joint>
+    <!-- RGB Camera -->
+    <link name="oak_rgb_camera_frame" />
+    <joint name="oak_rgb_camera_joint" type="fixed">
+        <parent link="oak" />
+        <child link="oak_rgb_camera_frame" />
+        <origin xyz="0 0 0" rpy="0 0 0" />
+    </joint>
+    <link name="oak_rgb_camera_optical_frame" />
+    <joint name="oak_rgb_camera_optical_joint" type="fixed">
+        <origin xyz="0 0 0" rpy="-1.57 0.0 -1.57" />
+        <parent link="oak_rgb_camera_frame" />
+        <child link="oak_rgb_camera_optical_frame" />
+    </joint>
+    <!-- Left Camera -->
+    <link name="oak_left_camera_frame" />
+    <joint name="oak_left_camera_joint" type="fixed">
+        <parent link="oak" />
+        <child link="oak_left_camera_frame" />
+        <origin xyz="0 0.0375 0" rpy="0 0 0" />
+    </joint>
+    <link name="oak_left_camera_optical_frame" />
+    <joint name="oak_left_camera_optical_joint" type="fixed">
+        <origin xyz="0 0 0" rpy="-1.57 0.0 -1.57" />
+        <parent link="oak_left_camera_frame" />
+        <child link="oak_left_camera_optical_frame" />
+    </joint>
+    <!-- right Camera -->
+    <link name="oak_right_camera_frame" />
+    <joint name="oak_right_camera_joint" type="fixed">
+        <parent link="oak" />
+        <child link="oak_right_camera_frame" />
+        <origin xyz="0 -0.0375 0" rpy="0 0 0" />
+    </joint>
+    <link name="oak_right_camera_optical_frame" />
+    <joint name="oak_right_camera_optical_joint" type="fixed">
+        <origin xyz="0 0 0" rpy="-1.57 0.0 -1.57" />
+        <parent link="oak_right_camera_frame" />
+        <child link="oak_right_camera_optical_frame" />
     </joint>
     <joint name="group_1_fastened_joint_63" type="fixed">
@@ -1776,5 +1829,5 @@
         <axis xyz="0 0 1" />
         <parent link="210000722" />
-        <child link="25085490_qt128光罩_v2_0a0" />
+        <child link="hesai_lidar" />
     </joint>
     <joint name="group_1_fastened_joint_8" type="fixed">

Commit message: Change OAK-D-W driver to v2. Fix problems with ros2_calib. First sensor calibration.

File: ros2_ws/bunker_description/urdf/sensors.urdf.xacro (robot description, xacro)
@@ -84,9 +84,9 @@
         <inertial>
             <mass value="3.54543e-05" />
-            <origin xyz="3.60929e-17 0.0325377 -8.29378e-18" rpy="0 -0 0" />
+            <origin xyz="3.60929e-17 0.0325377 -8.29378e-18" rpy="1.57 -0 0" />
             <inertia ixx="3.78835e-08" ixy="0" ixz="0" iyy="5.40715e-08" iyz="0" izz="3.78835e-08" />
         </inertial>
         <visual>
-            <origin xyz="0 0 0" rpy="0 -0 0" />
+            <origin xyz="0 0 0" rpy="1.57 -0 0" />
             <geometry>
                 <mesh filename="package://bunker_description/meshes/sensors/_25085490_QT128___V2_0A0.gltf" scale="1 1 1" />
@@ -116,9 +116,9 @@
         <inertial>
             <mass value="2.93529e-05" />
-            <origin xyz="1.71499e-10 -1.6419e-10 0.00273817" rpy="0 -0 0" />
+            <origin xyz="1.71499e-10 -1.6419e-10 0.00273817" rpy="-1.57 -0 0" />
             <inertia ixx="4.42717e-08" ixy="1.35997e-12" ixz="0" iyy="5.45764e-08" iyz="0" izz="9.78091e-08" />
         </inertial>
         <visual>
-            <origin xyz="0 0 0" rpy="0 -0 0" />
+            <origin xyz="0 0 0" rpy="-1.57 -0 0" />
             <geometry>
                 <mesh filename="package://bunker_description/meshes/sensors/_502_MFP0044.gltf" scale="1 1 1" />
@@ -588,5 +588,5 @@
         </inertial>
         <visual>
-            <origin xyz="0 0 0" rpy="0 -0 0" />
+            <origin xyz="0 0 0" rpy="-1.57 -0 -1.57" />
             <geometry>
                 <mesh filename="package://bunker_description/meshes/sensors/D_PRO_W_LENS_ADHESIVE_1.gltf" scale="1 1 1" />
@@ -1291,5 +1291,5 @@
         </inertial>
         <visual>
-            <origin xyz="0 0 0" rpy="0 -0 0" />
+            <origin xyz="0 0 0" rpy="1.57 0 -1.57" />
             <geometry>
                 <mesh filename="package://bunker_description/meshes/sensors/Top_Housing_MTi_630R_Casted_3_MTi_630R_MTi_6x0R_simple_2__MTi_6x0R_simple.gltf" scale="1 1 1" />
@@ -1358,4 +1358,5 @@
         <child link="part_1_3" />
     </joint>
+    # Aeva Atlas
     <joint name="fastened_3" type="fixed">
         <origin xyz="-0.066512 0.4015 0.026" rpy="1.5708 4.44089e-16 3.14159" />
@@ -1364,4 +1365,25 @@
         <child link="aeva/vehicle" />
     </joint>
+    <link name="aeva/ATLAS/sensor" />
+    <joint name="atlas_sensor_join" type="fixed">
+        <origin xyz="-0.066512 0.4015 0.026" rpy="1.5708 -1.57 3.14159" />
+        <axis xyz="0 -1 0" />
+        <parent link="aeva/vehicle" />
+        <child link="aeva/ATLAS/sensor" />
+    </joint>
+    <link name="aeva/ATLAS/camera" />
+    <joint name="atlas_camera_join" type="fixed">
+        <origin xyz="-0.066512 0.4015 0.026" rpy="1.5708 4.44089e-16 3.14159" />
+        <axis xyz="0 -1 0" />
+        <parent link="aeva/ATLAS/sensor" />
+        <child link="aeva/ATLAS/camera" />
+    </joint>
+    <link name="aeva/ATLAS/imu" />
+    <joint name="atlas_imu_join" type="fixed">
+        <origin xyz="-0.066512 0.4015 0.026" rpy="1.5708 4.44089e-16 3.14159" />
+        <axis xyz="0 -1 0" />
+        <parent link="aeva/ATLAS/sensor" />
+        <child link="aeva/ATLAS/imu" />
+    </joint>
     <joint name="fastened_4" type="fixed">
         <origin xyz="-0.075 0.027 0.051" rpy="-3.14159 -8.75812e-47 -2.73691e-48" />
@@ -1395,5 +1417,5 @@
     </joint>
     <joint name="group_1_fastened_joint" type="fixed">
-        <origin xyz="0.0375 0.0375 0.033" rpy="0 -0 0" />
+        <origin xyz="0.0375 0.0375 0.033" rpy="1.57 0.0 3.14" />
         <axis xyz="0 0 1" />
         <parent link="502_mfm0572" />
@@ -1485,5 +1507,5 @@
     </joint>
     <joint name="group_1_fastened_joint_22" type="fixed">
-        <origin xyz="-5.55112e-17 0 0" rpy="3.14159 -7.41768e-15 3.14159" />
+        <origin xyz="-5.55112e-17 0 0" rpy="-1.57 -1.57 0.0" />
         <axis xyz="0 0 1" />
         <parent link="_mti_6x0r_simple_2__mti_6x0r_simple_5" />
@@ -1682,73 +1704,73 @@
         <child link="cs2_62x_o_ring_20190509" />
     </joint>
+    <joint name="group_1_fastened_joint_53" type="fixed">
+        <origin xyz="0 0 0" rpy="0 -0 0" />
+        <axis xyz="0 0 1" />
+        <parent link="611_00020_16_1" />
+        <child link="612_00002_6" />
+    </joint>
+    <joint name="group_1_fastened_joint_54" type="fixed">
+        <origin xyz="0 0 0" rpy="0 -0 0" />
+        <axis xyz="0 0 1" />
+        <parent link="612_00002_6" />
+        <child link="612_00003_6" />
+    </joint>
+    <joint name="group_1_fastened_joint_55" type="fixed">
+        <origin xyz="0 0 0" rpy="0 -0 0" />
+        <axis xyz="0 0 1" />
+        <parent link="611_00016_20" />
+        <child link="611_00018_9" />
+    </joint>
+    <joint name="group_1_fastened_joint_56" type="fixed">
+        <origin xyz="-0.007 0.01175 0.013" rpy="0 -0 0" />
+        <axis xyz="0 0 1" />
+        <parent link="606_00014_02_5" />
+        <child link="611_00016_20" />
+    </joint>
+    <joint name="group_1_fastened_joint_57" type="fixed">
+        <origin xyz="0 0 0" rpy="0 -0 0" />
+        <axis xyz="0 0 1" />
+        <parent link="602_00007_1_3" />
+        <child link="602_00007_1_2" />
+    </joint>
+    <joint name="group_1_fastened_joint_58" type="fixed">
+        <origin xyz="0 0 0" rpy="0 -0 0" />
+        <axis xyz="0 0 1" />
+        <parent link="602_00007_1_1" />
+        <child link="602_00007_1" />
+    </joint>
+    <joint name="group_1_fastened_joint_59" type="fixed">
+        <origin xyz="0 0 0" rpy="0 -0 0" />
+        <axis xyz="0 0 1" />
+        <parent link="612_00003_6" />
+        <child link="cable_spacer" />
+    </joint>
+    <joint name="group_1_fastened_joint_6" type="fixed">
+        <origin xyz="0 -0.0824 0" rpy="0 1.85477e-122 0" />
+        <axis xyz="0 0 1" />
+        <parent link="黑色喷漆顶盖" />
+        <child link="210000722" />
+    </joint>
+    <joint name="group_1_fastened_joint_60" type="fixed">
+        <origin xyz="-0.007 0.01175 0.013" rpy="0 -0 0" />
+        <axis xyz="0 0 1" />
+        <parent link="606_00014_02_5" />
+        <child link="606_00013_02_6" />
+    </joint>
+    <joint name="group_1_fastened_joint_61" type="fixed">
+        <origin xyz="0 0 0" rpy="0 -0 0" />
+        <axis xyz="0 0 1" />
+        <parent link="602_00007_1_2" />
+        <child link="602_00007_1_1" />
+    </joint>
+    <!--OAK-D-W Camera-->
     <joint name="group_1_fastened_joint_52" type="fixed">
-        <origin xyz="0 0 0" rpy="0 -0 0" />
+        <origin xyz="0.008 0.13 0.0" rpy="1.57 -1.57 0" />
         <axis xyz="0 0 1" />
         <parent link="cable_spacer" />
         <child link="oak_parent_frame" />
     </joint>
-    <joint name="group_1_fastened_joint_53" type="fixed">
-        <origin xyz="0 0 0" rpy="0 -0 0" />
-        <axis xyz="0 0 1" />
-        <parent link="611_00020_16_1" />
-        <child link="612_00002_6" />
-    </joint>
-    <joint name="group_1_fastened_joint_54" type="fixed">
-        <origin xyz="0 0 0" rpy="0 -0 0" />
-        <axis xyz="0 0 1" />
-        <parent link="612_00002_6" />
-        <child link="612_00003_6" />
-    </joint>
-    <joint name="group_1_fastened_joint_55" type="fixed">
-        <origin xyz="0 0 0" rpy="0 -0 0" />
-        <axis xyz="0 0 1" />
-        <parent link="611_00016_20" />
-        <child link="611_00018_9" />
-    </joint>
-    <joint name="group_1_fastened_joint_56" type="fixed">
-        <origin xyz="-0.007 0.01175 0.013" rpy="0 -0 0" />
-        <axis xyz="0 0 1" />
-        <parent link="606_00014_02_5" />
-        <child link="611_00016_20" />
-    </joint>
-    <joint name="group_1_fastened_joint_57" type="fixed">
-        <origin xyz="0 0 0" rpy="0 -0 0" />
-        <axis xyz="0 0 1" />
-        <parent link="602_00007_1_3" />
-        <child link="602_00007_1_2" />
-    </joint>
-    <joint name="group_1_fastened_joint_58" type="fixed">
-        <origin xyz="0 0 0" rpy="0 -0 0" />
-        <axis xyz="0 0 1" />
-        <parent link="602_00007_1_1" />
-        <child link="602_00007_1" />
-    </joint>
-    <joint name="group_1_fastened_joint_59" type="fixed">
-        <origin xyz="0 0 0" rpy="0 -0 0" />
-        <axis xyz="0 0 1" />
-        <parent link="612_00003_6" />
-        <child link="cable_spacer" />
-    </joint>
-    <joint name="group_1_fastened_joint_6" type="fixed">
-        <origin xyz="0 -0.0824 0" rpy="0 1.85477e-122 0" />
-        <axis xyz="0 0 1" />
-        <parent link="黑色喷漆顶盖" />
-        <child link="210000722" />
-    </joint>
-    <joint name="group_1_fastened_joint_60" type="fixed">
-        <origin xyz="-0.007 0.01175 0.013" rpy="0 -0 0" />
-        <axis xyz="0 0 1" />
-        <parent link="606_00014_02_5" />
-        <child link="606_00013_02_6" />
-    </joint>
-    <joint name="group_1_fastened_joint_61" type="fixed">
-        <origin xyz="0 0 0" rpy="0 -0 0" />
-        <axis xyz="0 0 1" />
-        <parent link="602_00007_1_2" />
-        <child link="602_00007_1_1" />
-    </joint>
-    <!--OAK-D-W Camera-->
     <joint name="group_1_fastened_joint_62" type="fixed">
-        <origin xyz="0 0 0" rpy="0 0 1.57" />
+        <origin xyz="0 0 0" rpy="0 0 0" />
         <axis xyz="0 0 1" />
         <parent link="oak_parent_frame" />
@@ -1766,5 +1788,5 @@
         <child link="oak_imu_frame" />
         <origin xyz="0.0 -0.015 -0.013662"
-            rpy="0.0 1.57 0.0" />
+            rpy="0.0 1.57 3.14" />
     </joint>
     <!-- RGB Camera -->
@@ -1826,5 +1848,5 @@
     </joint>
     <joint name="group_1_fastened_joint_7" type="fixed">
-        <origin xyz="-1.57427e-08 0.0273 1.3773e-09" rpy="1.76983e-33 0.000181639 -1.23258e-32" />
+        <origin xyz="-1.57427e-08 0.0273 1.3773e-09" rpy="-1.57 4.71 0.0" /> <!--1.76983e-33 0.000181639 -1.23258e-32-->
         <axis xyz="0 0 1" />
         <parent link="210000722" />
