Commit message: prelim. simplified bunker description for testing

File: catkin_ws/src/bunker_description/urdf/sensors.urdf.xacro (robot description, xacro)
@@ -13,8 +13,8 @@
   <link name="imu" />
   <link name="radar_1" />
-  <link name="aeva/vehicle" />
+  <!-- <link name="aeva/vehicle" />
   <link name="aeva/ATLAS/sensor" />
   <link name="aeva/ATLAS/camera" />
-  <link name="aeva/ATLAS/imu" />
+  <link name="aeva/ATLAS/imu" /> -->
   <joint name="base_link_to_hesai_lidar_joint" type="fixed">
     <origin xyz="0.112963 0.0 0.388981" rpy="0.0008 0.000004 1.569201" />
