Commit message: glim working?

File: catkin_ws/src/PUTN/src/scout_simulator/scout_description/urdf/mini.xacro (robot description, xacro)
@@ -23,5 +23,5 @@
     <xacro:property name="wheel_radius" value="1.600e-01" />
     <!-- Base link -->
-    <link name="base_link">
+    <link name="aft_mapped">
         <visual>
             <origin
@@ -44,5 +44,5 @@
     <!-- <joint name="chassis_link_joint" type="fixed">
         <origin xyz="0 0 ${wheel_radius - wheel_vertical_offset}" rpy="0 0 0" />
-        <parent link="base_link" />
+        <parent link="aft_mapped" />
         <child link="chassis_link" />
     </joint> -->
@@ -56,5 +56,5 @@
     <joint name="inertial_joint" type="fixed">
         <origin xyz="0 0 0" rpy="0 0 0" />
-        <parent link="base_link" />
+        <parent link="aft_mapped" />
         <child link="inertial_link" />
     </joint>
@@ -64,5 +64,5 @@
         <origin xyz="0 0 0.5" rpy="0 0 0" />
         <parent link="world"/>
-        <child link="base_link"/>
+        <child link="aft_mapped"/>
     </joint> -->
     <!-- Scout wheel macros -->

File: catkin_ws/src/PUTN/src/scout_simulator/scout_description/urdf/scout_mini.urdf (robot description, URDF)
Before this commit: robot scout_mini, 6 links, 5 joints
Links:
- removed link base_link
- added link aft_mapped; collision mesh filename=package://scout_description/meshes/scout_mini_base_link2.dae; visual mesh filename=package://scout_description/meshes/scout_mini_base_link2.dae
Joints:
- joint front_left_wheel: parent base_link -> aft_mapped
- joint front_right_wheel: parent base_link -> aft_mapped
- joint inertial_joint: parent base_link -> aft_mapped
- joint rear_left_wheel: parent base_link -> aft_mapped
- joint rear_right_wheel: parent base_link -> aft_mapped

File: catkin_ws/src/PUTN/src/scout_simulator/scout_description/urdf/scout_mini.xacro (robot description, xacro)
@@ -23,5 +23,5 @@
     <xacro:property name="wheel_radius" value="1.600e-01" />
     <!-- Base link -->
-    <link name="base_link">
+    <link name="aft_mapped">
         <visual>
             <!--origin xyz="-0.0145261552504705 0.0231316650320557 0.00586280190939592" rpy="0 0 0" /-->
@@ -47,5 +47,5 @@
     <!-- <joint name="chassis_link_joint" type="fixed">
         <origin xyz="0 0 ${wheel_radius - wheel_vertical_offset}" rpy="0 0 0" />
-        <parent link="base_link" />
+        <parent link="aft_mapped" />
         <child link="chassis_link" />
     </joint> -->
@@ -72,5 +72,5 @@
     <joint name="inertial_joint" type="fixed">
         <origin xyz="0 0 0" rpy="0 0 0" />
-        <parent link="base_link" />
+        <parent link="aft_mapped" />
         <child link="inertial_link" />
     </joint>
@@ -80,5 +80,5 @@
         <origin xyz="0 0 0.5" rpy="0 0 0" />
         <parent link="world"/>
-        <child link="base_link"/>
+        <child link="aft_mapped"/>
     </joint> -->
     <!-- Scout wheel macros -->

File: catkin_ws/src/PUTN/src/scout_simulator/scout_description/urdf/scout_mini_wheel_1.xacro (robot description, xacro)
@@ -65,5 +65,5 @@
                   xyz="0.14547 0.20835 -0.07424"
                   rpy="0 1.57 0" />-->
-            <parent link="base_link"/>
+            <parent link="aft_mapped"/>
             <child link="${wheel_prefix}_wheel_link"/>
             <xacro:insert_block name="joint_pose"/>

File: catkin_ws/src/PUTN/src/scout_simulator/scout_description/urdf/scout_mini_wheel_2.xacro (robot description, xacro)
@@ -65,5 +65,5 @@
                   xyz="-0.17453 0.20835 -0.07424"
                   rpy="0 -1.57 0" />-->
-            <parent link="base_link"/>
+            <parent link="aft_mapped"/>
             <child link="${wheel_prefix}_wheel_link"/>
             <xacro:insert_block name="joint_pose"/>

File: catkin_ws/src/PUTN/src/scout_simulator/scout_description/urdf/scout_mini_wheel_3.xacro (robot description, xacro)
@@ -65,5 +65,5 @@
                   xyz="-0.17453 -0.24424 -0.07424"
                   rpy="0 -1.57 0" />-->
-            <parent link="base_link"/>
+            <parent link="aft_mapped"/>
             <child link="${wheel_prefix}_wheel_link"/>
             <xacro:insert_block name="joint_pose"/>

File: catkin_ws/src/PUTN/src/scout_simulator/scout_description/urdf/scout_mini_wheel_4.xacro (robot description, xacro)
@@ -65,5 +65,5 @@
                   xyz="0.19247 -0.24486 -0.073441"
                   rpy="-0 1.57 0" />-->
-            <parent link="base_link"/>
+            <parent link="aft_mapped"/>
             <child link="${wheel_prefix}_wheel_link"/>
             <xacro:insert_block name="joint_pose"/>

File: catkin_ws/src/PUTN/src/scout_simulator/scout_description/urdf/scout_v2.xacro (robot description, xacro)
@@ -7,5 +7,5 @@
     <xacro:include filename="$(find scout_description)/urdf/scout_wheel_type2.xacro" />
     <xacro:include filename="$(find velodyne_description)/urdf/HDL-32E.urdf.xacro"/>
-    <HDL-32E parent="base_link" name="velodyne" topic="/velodyne_points" hz="10" samples="440" gpu="false" lasers="32" max_range="100">
+    <HDL-32E parent="aft_mapped" name="velodyne" topic="/velodyne_points" hz="10" samples="440" gpu="false" lasers="32" max_range="100">
         <origin xyz="0 0 0.3" rpy="0 0 0" />
     </HDL-32E>
@@ -22,5 +22,5 @@
     <xacro:property name="wheel_radius" value="1.6459e-01" />
     <!-- Base link -->
-    <link name="base_link">
+    <link name="aft_mapped">
         <visual>
             <origin xyz="0 0 0" rpy="0 0 0" />
@@ -44,5 +44,5 @@
     <!-- <joint name="chassis_link_joint" type="fixed">
         <origin xyz="0 0 ${wheel_radius - wheel_vertical_offset}" rpy="0 0 0" />
-        <parent link="base_link" />
+        <parent link="aft_mapped" />
         <child link="chassis_link" />
     </joint> -->
@@ -59,5 +59,5 @@
     <joint name="inertial_joint" type="fixed">
         <origin xyz="0 0 0" rpy="0 0 0" />
-        <parent link="base_link" />
+        <parent link="aft_mapped" />
         <child link="inertial_link" />
     </joint>
@@ -67,5 +67,5 @@
         <origin xyz="0 0 0.5" rpy="0 0 0" />
         <parent link="world"/>
-        <child link="base_link"/>
+        <child link="aft_mapped"/>
     </joint> -->
     <!-- Scout wheel macros -->

File: catkin_ws/src/PUTN/src/scout_simulator/scout_description/urdf/scout_wheel_type1.xacro (robot description, xacro)
@@ -50,5 +50,5 @@
         </link>
         <joint name="${wheel_prefix}_wheel" type="continuous">
-            <parent link="base_link"/>
+            <parent link="aft_mapped"/>
             <child link="${wheel_prefix}_wheel_link"/>
             <xacro:insert_block name="joint_pose"/>

File: catkin_ws/src/PUTN/src/scout_simulator/scout_description/urdf/scout_wheel_type2.xacro (robot description, xacro)
@@ -50,5 +50,5 @@
         </link>
         <joint name="${wheel_prefix}_wheel" type="continuous">
-            <parent link="base_link"/>
+            <parent link="aft_mapped"/>
             <child link="${wheel_prefix}_wheel_link"/>
             <xacro:insert_block name="joint_pose"/>
