Commit message: ported ros1 ver bunker description

File: ros2_ws/src/bunker_packages/bunker_description/urdf/bunker.urdf.xacro (robot description, xacro)
@@ -28,5 +28,5 @@
       <geometry>
         <mesh
-          filename="package://bunker_description/meshes/base_link.STL" />
+          filename="package://bunker_description/meshes/bunker.STL" />
       </geometry>
       <material
@@ -42,5 +42,5 @@
       <geometry>
         <mesh
-          filename="package://bunker_description/meshes/base_link.STL" />
+          filename="package://bunker_description/meshes/bunker.STL" />
       </geometry>
     </collision>

File: ros2_ws/src/bunker_packages/bunker_description/urdf/sensors.urdf.xacro (robot description, xacro)
@@ -1,1886 +1,100 @@
 <?xml version="1.0" encoding="utf-8"?>
 <robot xmlns:xacro="http://www.ros.org/wiki/xacro">
-    <link name="20220058_耐落十字盘头螺钉_m2_6">
-        <inertial>
-            <mass value="2.60063e-08" />
-            <origin xyz="8.73996e-20 -0.00196618 -6.82502e-22" rpy="0 -0 0" />
-            <inertia ixx="7.8336e-14" ixy="0" ixz="0" iyy="3.31982e-14" iyz="0" izz="7.8336e-14" />
-        </inertial>
-        <visual>
-            <origin xyz="0 0 0" rpy="0 -0 0" />
-            <geometry>
-                <mesh filename="package://bunker_description/meshes/sensors/_20220058__________M2_6.gltf" scale="1 1 1" />
-            </geometry>
-            <material name="0.792157_0.819608_0.933333_0.000000_0.000000">
-                <color rgba="0.792157 0.819608 0.933333 1" />
-            </material>
-        </visual>
-    </link>
-    <link name="20220058_耐落十字盘头螺钉_m2_6_1">
-        <inertial>
-            <mass value="2.60063e-08" />
-            <origin xyz="8.73996e-20 -0.00196618 -6.82502e-22" rpy="0 -0 0" />
-            <inertia ixx="7.8336e-14" ixy="0" ixz="0" iyy="3.31982e-14" iyz="0" izz="7.8336e-14" />
-        </inertial>
-        <visual>
-            <origin xyz="0 0 0" rpy="0 -0 0" />
-            <geometry>
-                <mesh filename="package://bunker_description/meshes/sensors/_20220058__________M2_6.gltf" scale="1 1 1" />
-            </geometry>
-            <material name="0.792157_0.819608_0.933333_0.000000_0.000000">
-                <color rgba="0.792157 0.819608 0.933333 1" />
-            </material>
-        </visual>
-    </link>
-    <link name="20220058_耐落十字盘头螺钉_m2_6_2">
-        <inertial>
-            <mass value="2.60063e-08" />
-            <origin xyz="8.73996e-20 -0.00196618 -6.82502e-22" rpy="0 -0 0" />
-            <inertia ixx="7.8336e-14" ixy="0" ixz="0" iyy="3.31982e-14" iyz="0" izz="7.8336e-14" />
-        </inertial>
-        <visual>
-            <origin xyz="0 0 0" rpy="0 -0 0" />
-            <geometry>
-                <mesh filename="package://bunker_description/meshes/sensors/_20220058__________M2_6.gltf" scale="1 1 1" />
-            </geometry>
-            <material name="0.792157_0.819608_0.933333_0.000000_0.000000">
-                <color rgba="0.792157 0.819608 0.933333 1" />
-            </material>
-        </visual>
-    </link>
-    <link name="20220058_耐落十字盘头螺钉_m2_6_3">
-        <inertial>
-            <mass value="2.60063e-08" />
-            <origin xyz="8.73996e-20 -0.00196618 -6.82502e-22" rpy="0 -0 0" />
-            <inertia ixx="7.8336e-14" ixy="0" ixz="0" iyy="3.31982e-14" iyz="0" izz="7.8336e-14" />
-        </inertial>
-        <visual>
-            <origin xyz="0 0 0" rpy="0 -0 0" />
-            <geometry>
-                <mesh filename="package://bunker_description/meshes/sensors/_20220058__________M2_6.gltf" scale="1 1 1" />
-            </geometry>
-            <material name="0.792157_0.819608_0.933333_0.000000_0.000000">
-                <color rgba="0.792157 0.819608 0.933333 1" />
-            </material>
-        </visual>
-    </link>
-    <link name="210000722">
-        <inertial>
-            <mass value="5.0388e-05" />
-            <origin xyz="-0.000719833 0.00797759 0.00055236" rpy="0 -0 0" />
-            <inertia ixx="3.81257e-08" ixy="4.53901e-11" ixz="-1.82855e-10" iyy="6.69352e-08" iyz="1.65335e-10" izz="3.68438e-08" />
-        </inertial>
-        <visual>
-            <origin xyz="0 0 0" rpy="0 -0 0" />
-            <geometry>
-                <mesh filename="package://bunker_description/meshes/sensors/_210000722.gltf" scale="1 1 1" />
-            </geometry>
-            <material name="0.792157_0.819608_0.933333_0.000000_0.000000">
-                <color rgba="0.792157 0.819608 0.933333 1" />
-            </material>
-        </visual>
-    </link>
-    <link name="hesai_lidar">
-        <inertial>
-            <mass value="3.54543e-05" />
-            <origin xyz="3.60929e-17 0.0325377 -8.29378e-18" rpy="1.57 -0 0" />
-            <inertia ixx="3.78835e-08" ixy="0" ixz="0" iyy="5.40715e-08" iyz="0" izz="3.78835e-08" />
-        </inertial>
-        <visual>
-            <origin xyz="0 0 0" rpy="1.57 -0 0" />
-            <geometry>
-                <mesh filename="package://bunker_description/meshes/sensors/_25085490_QT128___V2_0A0.gltf" scale="1 1 1" />
-            </geometry>
-            <material name="0.082353_0.082353_0.082353_0.000000_0.000000">
-                <color rgba="0.0823529 0.0823529 0.0823529 1" />
-            </material>
-        </visual>
-    </link>
-    <link name="502_mfm0572">
-        <inertial>
-            <mass value="0.000138767" />
-            <origin xyz="0.0394159 0.0377686 0.0153731" rpy="0 -0 0" />
-            <inertia ixx="1.78561e-07" ixy="1.07361e-09" ixz="-5.77812e-10" iyy="2.22911e-07" iyz="2.94262e-10" izz="3.8789e-07" />
-        </inertial>
-        <visual>
-            <origin xyz="0.0375 0.0375 0.033" rpy="0 -0 0" />
-            <geometry>
-                <mesh filename="package://bunker_description/meshes/sensors/_502_MFM0572.gltf" scale="1 1 1" />
-            </geometry>
-            <material name="0.501961_0.501961_0.501961_0.000000_0.000000">
-                <color rgba="0.501961 0.501961 0.501961 1" />
-            </material>
-        </visual>
-    </link>
-    <link name="radar_1">
-        <inertial>
-            <mass value="2.93529e-05" />
-            <origin xyz="1.71499e-10 -1.6419e-10 0.00273817" rpy="-1.57 -0 0" />
-            <inertia ixx="4.42717e-08" ixy="1.35997e-12" ixz="0" iyy="5.45764e-08" iyz="0" izz="9.78091e-08" />
-        </inertial>
-        <visual>
-            <origin xyz="0 0 0" rpy="-1.57 -0 0" />
-            <geometry>
-                <mesh filename="package://bunker_description/meshes/sensors/_502_MFP0044.gltf" scale="1 1 1" />
-            </geometry>
-            <material name="0.109804_0.109804_0.109804_0.000000_0.000000">
-                <color rgba="0.109804 0.109804 0.109804 1" />
-            </material>
-        </visual>
-    </link>
-    <link name="600_13737_0000_a01">
-        <inertial>
-            <mass value="1.71817e-05" />
-            <origin xyz="0.0481466 0.0419946 0.000785" rpy="0 -0 0" />
-            <inertia ixx="1.58366e-08" ixy="-6.40503e-12" ixz="0" iyy="1.5926e-08" iyz="0" izz="3.17555e-08" />
-        </inertial>
-        <visual>
-            <origin xyz="0 0 0" rpy="0 -0 0" />
-            <geometry>
-                <mesh filename="package://bunker_description/meshes/sensors/_600_13737_0000_A01.gltf" scale="1 1 1" />
-            </geometry>
-            <material name="0.498039_0.498039_0.498039_0.000000_0.000000">
-                <color rgba="0.498039 0.498039 0.498039 1" />
-            </material>
-        </visual>
-    </link>
-    <link name="602_00007_1">
-        <inertial>
-            <mass value="6.43779e-08" />
-            <origin xyz="0.0695091 -0.0219904 -0.00223951" rpy="0 -0 0" />
-            <inertia ixx="6.54799e-13" ixy="0" ixz="0" iyy="6.54841e-13" iyz="0" izz="1.13714e-13" />
-        </inertial>
-        <visual>
-            <origin xyz="0 0 0" rpy="0 -0 0" />
-            <geometry>
-                <mesh filename="package://bunker_description/meshes/sensors/_602_00007_1.gltf" scale="1 1 1" />
-            </geometry>
-            <material name="0.980392_0.713725_0.003922_0.000000_0.000000">
-                <color rgba="0.980392 0.713726 0.00392157 1" />
-            </material>
-        </visual>
-    </link>
-    <link name="602_00007_1_1">
-        <inertial>
-            <mass value="6.43779e-08" />
-            <origin xyz="0.0183491 -0.0219904 -0.00223951" rpy="0 -0 0" />
-            <inertia ixx="6.54799e-13" ixy="0" ixz="0" iyy="6.54841e-13" iyz="0" izz="1.13714e-13" />
-        </inertial>
-        <visual>
-            <origin xyz="0 0 0" rpy="0 -0 0" />
-            <geometry>
-                <mesh filename="package://bunker_description/meshes/sensors/_602_00007_1_1.gltf" scale="1 1 1" />
-            </geometry>
-            <material name="0.615686_0.811765_0.929412_0.000000_0.000000">
-                <color rgba="0.615686 0.811765 0.929412 1" />
-            </material>
-        </visual>
-    </link>
-    <link name="602_00007_1_2">
-        <inertial>
-            <mass value="6.43779e-08" />
-            <origin xyz="0.0737991 -0.00350039 -0.00223951" rpy="0 -0 0" />
-            <inertia ixx="6.54799e-13" ixy="0" ixz="0" iyy="6.54841e-13" iyz="0" izz="1.13714e-13" />
-        </inertial>
-        <visual>
-            <origin xyz="0 0 0" rpy="0 -0 0" />
-            <geometry>
-                <mesh filename="package://bunker_description/meshes/sensors/_602_00007_1_2.gltf" scale="1 1 1" />
-            </geometry>
-            <material name="0.647059_0.647059_0.647059_0.000000_0.000000">
-                <color rgba="0.647059 0.647059 0.647059 1" />
-            </material>
-        </visual>
-    </link>
-    <link name="602_00007_1_3">
-        <inertial>
-            <mass value="6.43779e-08" />
-            <origin xyz="0.0157491 -0.00350039 -0.00223951" rpy="0 -0 0" />
-            <inertia ixx="6.54799e-13" ixy="0" ixz="0" iyy="6.54841e-13" iyz="0" izz="1.13714e-13" />
-        </inertial>
-        <visual>
-            <origin xyz="0 0 0" rpy="0 -0 0" />
-            <geometry>
-                <mesh filename="package://bunker_description/meshes/sensors/_602_00007_1_3.gltf" scale="1 1 1" />
-            </geometry>
-            <material name="0.231373_0.380392_0.705882_0.000000_0.000000">
-                <color rgba="0.231373 0.380392 0.705882 1" />
-            </material>
-        </visual>
-    </link>
-    <link name="606_00013_02_6">
-        <inertial>
-            <mass value="5.28711e-06" />
-            <origin xyz="0.04443 -0.0117643 0.00756731" rpy="0 -0 0" />
-            <inertia ixx="4.5871e-10" ixy="1.52284e-12" ixz="1.30136e-11" iyy="4.24249e-09" iyz="1.19905e-11" izz="4.67221e-09" />
-        </inertial>
-        <visual>
-            <origin xyz="0 0 0" rpy="0 -0 0" />
-            <geometry>
-                <mesh filename="package://bunker_description/meshes/sensors/_606_00013_02_6.gltf" scale="1 1 1" />
-            </geometry>
-            <material name="0.972549_0.529412_0.003922_0.000000_0.000000">
-                <color rgba="0.972549 0.529412 0.00392157 1" />
-            </material>
-        </visual>
-    </link>
-    <link name="606_00014_02_5">
-        <inertial>
-            <mass value="2.06767e-05" />
-            <origin xyz="0.0373269 0.000131764 0.00910485" rpy="0 -0 0" />
-            <inertia ixx="2.05318e-09" ixy="-8.59665e-11" ixz="-1.34501e-11" iyy="1.66385e-08" iyz="-1.59785e-11" izz="1.77983e-08" />
-        </inertial>
-        <visual>
-            <origin xyz="-0.007 0.01175 0.013" rpy="0 -0 0" />
-            <geometry>
-                <mesh filename="package://bunker_description/meshes/sensors/_606_00014_02_5.gltf" scale="1 1 1" />
-            </geometry>
-            <material name="0.498039_0.498039_0.498039_0.000000_0.000000">
-                <color rgba="0.498039 0.498039 0.498039 1" />
-            </material>
-        </visual>
-    </link>
-    <link name="611_00016_20">
-        <inertial>
-            <mass value="9.82365e-08" />
-            <origin xyz="0.0632437 -0.00704037 0.0023009" rpy="0 -0 0" />
-            <inertia ixx="1.28378e-12" ixy="0" ixz="0" iyy="2.7916e-12" iyz="0" izz="4.03347e-12" />
-        </inertial>
-        <visual>
-            <origin xyz="0 0 0" rpy="0 -0 0" />
-            <geometry>
-                <mesh filename="package://bunker_description/meshes/sensors/_611_00016_20.gltf" scale="1 1 1" />
-            </geometry>
-            <material name="0.647059_0.647059_0.647059_0.000000_0.000000">
-                <color rgba="0.647059 0.647059 0.647059 1" />
-            </material>
-        </visual>
-    </link>
-    <link name="611_00018_9">
-        <inertial>
-            <mass value="1.98811e-07" />
-            <origin xyz="0.0445 -0.00698625 0.0063509" rpy="0 -0 0" />
-            <inertia ixx="3.5467e-12" ixy="0" ixz="0" iyy="3.5467e-12" iyz="0" izz="6.88631e-12" />
-        </inertial>
-        <visual>
-            <origin xyz="0 0 0" rpy="0 -0 0" />
-            <geometry>
-                <mesh filename="package://bunker_description/meshes/sensors/_611_00018_9.gltf" scale="1 1 1" />
-            </geometry>
-            <material name="0.768627_0.886275_0.952941_0.000000_0.000000">
-                <color rgba="0.768627 0.886275 0.952941 1" />
-            </material>
-        </visual>
-    </link>
-    <link name="611_00020_16_1">
-        <inertial>
-            <mass value="2.5919e-07" />
-            <origin xyz="0.082 -0.00698622 0.0066009" rpy="0 -0 0" />
-            <inertia ixx="4.52365e-12" ixy="0" ixz="0" iyy="4.52365e-12" iyz="0" izz="8.65852e-12" />
-        </inertial>
-        <visual>
-            <origin xyz="0 0 0" rpy="0 -0 0" />
-            <geometry>
-                <mesh filename="package://bunker_description/meshes/sensors/_611_00020_16_1.gltf" scale="1 1 1" />
-            </geometry>
-        </visual>
-    </link>
-    <link name="611_00020_16__1_">
-        <inertial>
-            <mass value="1e-09" />
-            <origin xyz="0 0 0" rpy="0 -0 0" />
-            <inertia ixx="4e-14" ixy="0" ixz="0" iyy="4e-14" iyz="0" izz="4e-14" />
-        </inertial>
-    </link>
-    <link name="612_00002_6">
-        <inertial>
-            <mass value="5e-08" />
-            <origin xyz="0.03043 -0.01299 -0.00105" rpy="0 -0 0" />
-            <inertia ixx="4.17708e-13" ixy="0" ixz="0" iyy="4.17708e-13" iyz="0" izz="8.33333e-13" />
-        </inertial>
-        <visual>
-            <origin xyz="0 0 0" rpy="0 -0 0" />
-            <geometry>
-                <mesh filename="package://bunker_description/meshes/sensors/_612_00002_6.gltf" scale="1 1 1" />
-            </geometry>
-            <material name="0.498039_0.498039_0.498039_0.000000_0.000000">
-                <color rgba="0.498039 0.498039 0.498039 1" />
-            </material>
-        </visual>
-    </link>
-    <link name="612_00003_6">
-        <inertial>
-            <mass value="4.95e-07" />
-            <origin xyz="0.0585 -0.008 -0.00055" rpy="0 -0 0" />
-            <inertia ixx="9.37406e-12" ixy="0" ixz="0" iyy="2.00578e-11" iyz="0" izz="2.92463e-11" />
-        </inertial>
-        <visual>
-            <origin xyz="0 0 0" rpy="0 -0 0" />
-            <geometry>
-                <mesh filename="package://bunker_description/meshes/sensors/_612_00003_6.gltf" scale="1 1 1" />
-            </geometry>
-            <material name="0.972549_0.529412_0.003922_0.000000_0.000000">
-                <color rgba="0.972549 0.529412 0.00392157 1" />
-            </material>
-        </visual>
-    </link>
-    <link name="_mti_6x0r_simple_2__mti_6x0r_simple">
-        <inertial>
-            <mass value="1.94005e-10" />
-            <origin xyz="0.00654955 0.024755 0.000743914" rpy="0 -0 0" />
-            <inertia ixx="0" ixy="0" ixz="0" iyy="0" iyz="0" izz="0" />
-        </inertial>
-        <visual>
-            <origin xyz="0 0 0" rpy="0 -0 0" />
-            <geometry>
-                <mesh filename="package://bunker_description/meshes/sensors/_MTi_6x0R_simple_2__MTi_6x0R_simple.gltf" scale="1 1 1" />
-            </geometry>
-            <material name="0.917647_0.407843_0.321569_0.000000_0.000000">
-                <color rgba="0.917647 0.407843 0.321569 1" />
-            </material>
-        </visual>
-    </link>
-    <link name="_mti_6x0r_simple_2__mti_6x0r_simple_1">
-        <inertial>
-            <mass value="1.59726e-10" />
-            <origin xyz="-0.00685629 0.024755 0.0011395" rpy="0 -0 0" />
-            <inertia ixx="0" ixy="0" ixz="0" iyy="1.03503e-15" iyz="0" izz="0" />
-        </inertial>
-        <visual>
-            <origin xyz="0 0 0" rpy="0 -0 0" />
-            <geometry>
-                <mesh filename="package://bunker_description/meshes/sensors/_MTi_6x0R_simple_2__MTi_6x0R_simple_1.gltf" scale="1 1 1" />
-            </geometry>
-            <material name="0.917647_0.407843_0.321569_0.000000_0.000000">
-                <color rgba="0.917647 0.407843 0.321569 1" />
-            </material>
-        </visual>
-    </link>
-    <link name="_mti_6x0r_simple_2__mti_6x0r_simple_2">
-        <inertial>
-            <mass value="1.96917e-10" />
-            <origin xyz="-0.013421 0.024755 0.000677911" rpy="0 -0 0" />
-            <inertia ixx="0" ixy="0" ixz="0" iyy="1.01315e-15" iyz="0" izz="0" />
-        </inertial>
-        <visual>
-            <origin xyz="0 0 0" rpy="0 -0 0" />
-            <geometry>
-                <mesh filename="package://bunker_description/meshes/sensors/_MTi_6x0R_simple_2__MTi_6x0R_simple_2.gltf" scale="1 1 1" />
-            </geometry>
-            <material name="0.917647_0.407843_0.321569_0.000000_0.000000">
-                <color rgba="0.917647 0.407843 0.321569 1" />
-            </material>
-        </visual>
-    </link>
-    <link name="_mti_6x0r_simple_2__mti_6x0r_simple_3">
-        <inertial>
-            <mass value="7.72548e-11" />
-            <origin xyz="0.0141036 0.024755 0.000715696" rpy="0 -0 0" />
-            <inertia ixx="0" ixy="0" ixz="0" iyy="0" iyz="0" izz="0" />
-        </inertial>
-        <visual>
-            <origin xyz="0 0 0" rpy="0 -0 0" />
-            <geometry>
-                <mesh filename="package://bunker_description/meshes/sensors/_MTi_6x0R_simple_2__MTi_6x0R_simple_3.gltf" scale="1 1 1" />
-            </geometry>
-            <material name="0.917647_0.407843_0.321569_0.000000_0.000000">
-                <color rgba="0.917647 0.407843 0.321569 1" />
-            </material>
-        </visual>
-    </link>
-    <link name="_mti_6x0r_simple_2__mti_6x0r_simple_4">
-        <inertial>
-            <mass value="2.25801e-10" />
-            <origin xyz="-5.09875e-05 0.024755 0.00075991" rpy="0 -0 0" />
-            <inertia ixx="0" ixy="0" ixz="0" iyy="1.22058e-15" iyz="0" izz="0" />
-        </inertial>
-        <visual>
-            <origin xyz="0 0 0" rpy="0 -0 0" />
-            <geometry>
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